Commit message: v2.0: fill-based approach, place dock, known-cube scan/creep.
Drive forward until grasp-box fill is large enough (not cy/err_u alone); keep place front dock, FOV-safe creep, and map scan when cube is intermittent.

File: mybot_description/urdf/arm_gazebo.xacro (robot description, xacro)
@@ -31,9 +31,9 @@
         <material>Gazebo/White</material>
     </gazebo>
-    <xacro:macro name="ros2_control_joint" params="joint_name">
+    <xacro:macro name="ros2_control_joint" params="joint_name min:=-3.14 max:=3.14">
         <joint name="${joint_name}">
             <command_interface name="position">
-                <param name="min">-1</param>
-                <param name="max">1</param>
+                <param name="min">${min}</param>
+                <param name="max">${max}</param>
             </command_interface>
             <state_interface name="position">
@@ -47,12 +47,13 @@
             <plugin>gazebo_ros2_control/GazeboSystem</plugin>
         </hardware>
+        <!-- Was wrongly ±1 → PICK j2/j3≈1.15 rejected, arm stayed up -->
         <xacro:ros2_control_joint joint_name="joint1" />
-        <xacro:ros2_control_joint joint_name="joint2" />
-        <xacro:ros2_control_joint joint_name="joint3" />
+        <xacro:ros2_control_joint joint_name="joint2" min="-2.35" max="2.35" />
+        <xacro:ros2_control_joint joint_name="joint3" min="-2.62" max="2.62" />
         <xacro:ros2_control_joint joint_name="joint4" />
-        <xacro:ros2_control_joint joint_name="joint5" />
+        <xacro:ros2_control_joint joint_name="joint5" min="-2.35" max="2.35" />
         <xacro:ros2_control_joint joint_name="joint6" />
-        <xacro:ros2_control_joint joint_name="finger_joint1" />
-        <xacro:ros2_control_joint joint_name="finger_joint2" />
+        <xacro:ros2_control_joint joint_name="finger_joint1" min="0.0" max="0.08" />
+        <xacro:ros2_control_joint joint_name="finger_joint2" min="0.0" max="0.08" />
     </ros2_control>
     <!-- gazebo_ros2_contril -->

File: mybot_description/urdf/large_base.xacro (robot description, xacro)
@@ -5,10 +5,12 @@
     <!-- PROPERTY LIST -->
     <xacro:property name="M_PI" value="3.1415926" />
-    <xacro:property name="base_mass" value="2" />
+    <!-- Original lighter chassis (was 28 kg for anti-fly; user testing feel) -->
+    <!-- Heavier again: tip/fly when driving over placed cubes with 2 kg -->
+    <xacro:property name="base_mass" value="18" />
     <xacro:property name="base_width" value="0.320" />
     <xacro:property name="base_length" value="0.320" />
     <xacro:property name="base_height" value="0.1" />
     <!-- 轮子 -->
-    <xacro:property name="wheel_mass" value="0.4" />
+    <xacro:property name="wheel_mass" value="0.5" />
     <xacro:property name="wheel_radius" value="0.065" />
     <xacro:property name="wheel_length" value="0.050" />
@@ -55,7 +57,7 @@
     </xacro:macro>
     <!-- Macro for robot 轮子 -->
-    <xacro:macro name="wheel" params="prefix reflect">
+    <xacro:macro name="wheel" params="prefix reflect x:=${wheel_joint_x}">
         <joint name="${prefix}_wheel_joint" type="continuous">
-            <origin xyz="${wheel_joint_x} ${reflect*(base_width+wheel_length)/2} ${-wheel_joint_z}"
+            <origin xyz="${x} ${reflect*(base_width+wheel_length)/2} ${-wheel_joint_z}"
                 rpy="0 0 0" />
             <parent link="base_link" />
@@ -136,4 +138,5 @@
             h="${base_height}" />
     </link>
+    <!-- 2 driven wheels + rear caster only (known-good Gazebo baseline) -->
     <xacro:wheel prefix="left" reflect="1" />
     <xacro:wheel prefix="right" reflect="-1" />

File: mybot_description/urdf/large_base_gazebo.xacro (robot description, xacro)
@@ -32,5 +32,5 @@
     <xacro:wheel_transmission prefix="left" />
     <xacro:wheel_transmission prefix="right" />
-    <!-- controller -->
+    <!-- Restored known-good 2-wheel diff drive (matches pre-4WD backup) -->
     <gazebo>
         <plugin name="differential_drive_controller" filename="libgazebo_ros_diff_drive.so">
@@ -40,19 +40,18 @@
             <wheel_separation>${wheel_joint_y*2}</wheel_separation>
             <wheel_diameter>${2*wheel_radius}</wheel_diameter>
-            <max_wheel_torque>10</max_wheel_torque>
-            <max_wheel_acceleration>1.0</max_wheel_acceleration>
+            <!-- mass≈18 needs more torque than backup's 10 -->
+            <max_wheel_torque>35</max_wheel_torque>
+            <max_wheel_acceleration>1.5</max_wheel_acceleration>
             <command_topic>cmd_vel</command_topic>
             <publish_odom>true</publish_odom>
-            <!-- Only EKF publishes odom→base_footprint TF (avoid dual TF drift). -->
+            <!-- Only EKF publishes odom→base_footprint TF -->
             <publish_odom_tf>false</publish_odom_tf>
-            <publish_wheel_tf>true</publish_wheel_tf>
+            <publish_wheel_tf>false</publish_wheel_tf>
             <odometry_topic>odom</odometry_topic>
             <odometry_frame>odom</odometry_frame>
             <robot_base_frame>base_footprint</robot_base_frame>
             <odometry_source>1</odometry_source>
-	    <!-- 强制 2D 位姿，Z 轴恒为 0 -->
-	    <odometry_2d_only>true</odometry_2d_only>
-	    <!-- 或者使用下面这个参数（不同版本可能不同） -->
-	    <publish_odom_2d_only>true</publish_odom_2d_only>
+            <odometry_2d_only>true</odometry_2d_only>
+            <publish_odom_2d_only>true</publish_odom_2d_only>
         </plugin>
     </gazebo>
