Commit message: v12: compact cube/zone layout, GT localization, smoother pick nav.
Pull A/B/C and cubes closer, fix blue/red approach sides, allow DWB reverse and slower replan so pick nav stops crawling in reverse.

Co-authored-by: Cursor <cursoragent@cursor.com>

File: mybot_description/urdf/large_base.xacro (robot description, xacro)
@@ -17,5 +17,6 @@
     <xacro:property name="wheel_joint_x" value="0.14" />
     <xacro:property name="wheel_joint_y" value="0.38" />
-    <xacro:property name="wheel_joint_z" value="0.035" />
+    <!-- 比万向轮着地点低约 2 mm，直线时驱动轮吃到重量。0.035 时轮底悬空，只有转弯压轮才快 -->
+    <xacro:property name="wheel_joint_z" value="0.040" />
     <!-- 支撑轮 -->
     <xacro:property name="caster_mass" value="0.4" />

File: mybot_description/urdf/large_base_gazebo.xacro (robot description, xacro)
@@ -29,4 +29,7 @@
     <gazebo reference="back_caster_link">
         <material>Gazebo/Black</material>
+        <!-- 固定球没有转向轴，摩擦一大，过弯会把前进速度拖掉 -->
+        <mu1>0.05</mu1>
+        <mu2>0.05</mu2>
     </gazebo>
     <xacro:wheel_transmission prefix="left" />
@@ -38,9 +41,10 @@
             <left_joint>left_wheel_joint</left_joint>
             <right_joint>right_wheel_joint</right_joint>
-            <wheel_separation>${wheel_joint_y*2}</wheel_separation>
+            <!-- 左右轮中心距，不用 wheel_joint_y*2（那是 0.76，实际只有 0.37，转弯会差一倍） -->
+            <wheel_separation>${base_width + wheel_length}</wheel_separation>
             <wheel_diameter>${2*wheel_radius}</wheel_diameter>
-            <!-- mass≈18 needs more torque than backup's 10 -->
             <max_wheel_torque>35</max_wheel_torque>
-            <max_wheel_acceleration>1.5</max_wheel_acceleration>
+            <!-- 线加速度 m/s²。4 时两轮一起加速爬不到直线指令，转弯单轮差速反而显得快 -->
+            <max_wheel_acceleration>10.0</max_wheel_acceleration>
             <command_topic>cmd_vel</command_topic>
             <publish_odom>true</publish_odom>
